File: Amplificador/pcb_amplificador/pcb_amplificador.kicad_pcb (KiCad board)
At the start: 2 copper layers, 123 parts, among them CON1 SJ-3523-SMT-TR, J1 Screw_Terminal_01x02, J2 Conn_01x03_Male, J3 Screw_Terminal_01x06, K1 SANYOU_SRD_Form_B, M1 FDS9934C, M2 FDS9934C, M3 FDS9934C, Q1 BC860, Q10 BD139, Q11 BD140, Q12 BD139, Q13 2SA1943-O_Q_, Q14 2SC5200-O_Q, Q15 2SA1943-O_Q_, Q16 2SC5200-O_Q, Q17 2SAR514P5, Q18 BC860, Q19 BC860, Q2 BC860, Q20 2SAR514P5, Q21 2SCR514P5, Q22 2SCR514P5, Q23 2SCR514P5, Q24 2SAR514P5, Q25 2SCR514P5, Q26 BC817, Q27 BC817, Q28 BC807, Q3 BC850, Q4 BC850, Q5 BC860, Q6 BC860, Q7 BC850, Q8 2SCR514P5, Q9 2SCR514P5

Commit message: Avance con el PCB
Parts:
- added R9: 0, Resistor_SMD:R_1206_3216Metric_Pad1.42x1.75mm_HandSolder, F.Cu at (62.7, 80.6)
- R21: footprint Resistor_SMD:R_0815_2038Metric_Pad1.53x4.00mm_HandSolder -> Resistor_SMD:R_0805_2012Metric_Pad1.15x1.40mm_HandSolder
- moved Q10 116.9 mm to (102.0, 63.2), turned to 90 degrees
- moved R7 116.7 mm to (57.4, 90.0), turned to 270 degrees
- moved C4 115.5 mm to (55.7, 83.1), turned to 180 degrees
- moved R8 111.9 mm to (62.3, 92.2), turned to 90 degrees
- moved RV1 110.5 mm to (102.7, 68.8)
- moved Q7 108.9 mm to (55.8, 86.1), turned to 180 degrees
- moved C6 102.6 mm to (108.3, 62.2)
- moved Q25 100.9 mm to (65.7, 85.2), turned to 90 degrees
- moved C5 100.4 mm to (55.0, 90.8), turned to 90 degrees
- moved Q8 88.5 mm to (60.1, 85.3), turned to 90 degrees
- moved R17 81.9 mm to (75.4, 53.7), turned to 90 degrees
- moved R13 81.3 mm to (106.8, 54.5)
- moved R10 80.8 mm to (97.9, 58.1), turned to 270 degrees
- moved R44 78.9 mm to (60.5, 88.9), turned to 180 degrees
- moved C7 77.8 mm to (62.7, 56.7), turned to 270 degrees
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Connections:
- C6 pad 1: Net-(C4-Pad1) -> Net-(C6-Pad1)
- Q10 pad 1: Net-(C4-Pad1) -> Net-(C6-Pad1)
- Q18 pad 3: Net-(Q17-Pad3) -> Net-(Q17-Pad1)
- Q19 pad 1: Net-(Q17-Pad3) -> Net-(Q17-Pad1)
- Q20 pad 1: Net-(D5-Pad1) -> Net-(D7-Pad1)
- Q20 pad 3: Net-(D7-Pad1) -> Net-(D5-Pad1)
- Q21 pad 1: Net-(D11-Pad2) -> Net-(D13-Pad2)
- Q21 pad 2: Net-(D13-Pad2) -> Net-(D13-Pad1)
- Q21 pad 3: Net-(D13-Pad1) -> Net-(D11-Pad2)
- Q22 pad 1: Net-(D12-Pad1) -> Net-(Q22-Pad1)
- Q22 pad 2: Net-(Q22-Pad2) -> Net-(D22-Pad2)
- Q22 pad 3: Net-(D22-Pad2) -> Net-(D12-Pad1)
- Q23 pad 1: /-Vmax -> Net-(Q11-Pad2)
- Q23 pad 2: Net-(Q11-Pad2) -> Net-(D9-Pad2)
- Q23 pad 3: Net-(D9-Pad2) -> /-Vmax
- Q24 pad 1: /Vmax -> Net-(Q12-Pad2)
- Q24 pad 3: Net-(Q12-Pad2) -> /Vmax
- Q25 pad 1: Net-(C5-Pad1) -> Net-(Q25-Pad1)
- Q25 pad 2: Net-(Q25-Pad2) -> Net-(C4-Pad2)
- Q25 pad 3: Net-(C4-Pad2) -> Net-(C5-Pad1)
- Q8 pad 1: Net-(Q8-Pad1) -> Net-(Q7-Pad2)
- Q8 pad 2: Net-(Q7-Pad2) -> Net-(C4-Pad1)
- Q8 pad 3: Net-(C4-Pad1) -> Net-(Q8-Pad3)
- Q9 pad 1: Net-(D12-Pad1) -> Net-(Q9-Pad1)
- Q9 pad 2: Net-(Q9-Pad2) -> Net-(D21-Pad1)
- Q9 pad 3: Net-(D21-Pad1) -> Net-(D12-Pad1)
- R11 pad 2: Net-(C4-Pad1) -> Net-(C6-Pad1)
- R15 pad 2: Net-(Q9-Pad2) -> Net-(Q9-Pad1)
- R16 pad 2: Net-(Q9-Pad2) -> Net-(Q9-Pad1)
- R17 pad 1: Net-(Q17-Pad1) -> Net-(Q17-Pad3)
- R18 pad 1: Net-(Q17-Pad1) -> Net-(Q17-Pad3)
- R20 pad 1: Net-(Q17-Pad3) -> Net-(Q17-Pad1)
- R37 pad 1: Net-(Q9-Pad2) -> Net-(Q9-Pad1)
- R38 pad 1: Net-(Q22-Pad2) -> Net-(Q22-Pad1)
- R39 pad 2: Net-(Q22-Pad2) -> Net-(Q22-Pad1)
- R40 pad 2: Net-(Q22-Pad2) -> Net-(Q22-Pad1)
- R43 pad 1: Net-(Q8-Pad1) -> Net-(Q8-Pad3)
- R43 pad 2: Net-(Q25-Pad2) -> Net-(Q25-Pad1)
- R44 pad 1: Net-(Q8-Pad1) -> Net-(Q8-Pad3)
- RV1 pad 1: Net-(C4-Pad1) -> Net-(C6-Pad1)
- RV1 pad 2: Net-(C4-Pad1) -> Net-(C6-Pad1)
Routing:
- net Net-(C7-Pad2): track 0.00 -> 54.0 mm
- net Net-(Q17-Pad1): track 0.00 -> 35.3 mm
- net Net-(C5-Pad1): track 2.03 -> 33.4 mm
- net Earth: track 0.00 -> 22.4 mm, vias 0 -> 5
- net Net-(C4-Pad2): track 3.70 -> 24.4 mm
- net Net-(C1-Pad2): track 0.36 -> 17.3 mm
- net Net-(CON1-Pad3): track 0.00 -> 12.2 mm
- net Net-(C7-Pad1): track 0.00 -> 11.7 mm
- net Net-(Q17-Pad3): track 0.00 -> 11.2 mm
- net Net-(C4-Pad1): track 0.00 -> 6.27 mm
- net Net-(Q7-Pad2): track 0.00 -> 5.61 mm
- net Net-(Q8-Pad3): track 0.00 -> 4.80 mm
- net Net-(Q19-Pad3): track 0.00 -> 4.20 mm
- net Net-(C2-Pad2): track 24.3 -> 28.1 mm
- net Net-(Q25-Pad1): track 0.00 -> 3.31 mm
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
Commit message: Avance PCB
Parts:
- RV1: footprint Potentiometer_THT:Potentiometer_Bourns_3296W_Vertical -> Potentiometer_SMD:Potentiometer_Bourns_3314G_Vertical
- moved K1 195.8 mm to (133.3, 104.8)
- moved C12 187.6 mm to (141.6, 128.3), turned to 270 degrees
- moved C14 186.8 mm to (149.2, 128.3), turned to 270 degrees
- moved J1 172.0 mm to (158.1, 102.9), turned to 270 degrees
- moved C13 171.5 mm to (141.6, 119.4)
- moved M3 171.3 mm to (149.9, 119.4)
- moved C8 161.3 mm to (77.0, 132.3)
- moved D18 154.3 mm to (81.0, 122.7), turned to 90 degrees
- moved R51 152.7 mm to (131.4, 123.2), turned to 180 degrees
- moved Q16 151.1 mm to (104.9, 93.7), turned to 180 degrees
- moved Q27 150.2 mm to (135.3, 130.2), turned to 270 degrees
- moved R46 148.6 mm to (136.5, 122.2), turned to 90 degrees
- moved R45 146.6 mm to (136.5, 126.4), turned to 270 degrees
- moved D20 146.6 mm to (83.6, 122.7), turned to 270 degrees
- moved Q28 146.0 mm to (131.4, 130.2), turned to 180 degrees
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Connections:
- net Net-(D12-Pad1) renamed /VOUT
Routing:
- net Net-(D17-Pad2): track 2.41 -> 48.6 mm
- net Net-(C7-Pad2): track 54.0 -> 17.5 mm
- net Net-(C6-Pad2): track 0.00 -> 20.8 mm
- net Net-(C6-Pad1): track 0.00 -> 19.7 mm
- net Net-(C13-Pad1): track 0.00 -> 17.1 mm
- net Net-(Q10-Pad3): track 0.00 -> 13.4 mm
- net Net-(Q17-Pad1): track 35.3 -> 26.2 mm
- net Net-(C3-Pad1): track 0.00 -> 8.68 mm
- net Net-(C12-Pad1): track 0.00 -> 7.76 mm
- net Net-(C12-Pad2): track 0.00 -> 7.62 mm
- net Net-(Q26-Pad1): track 0.00 -> 7.39 mm
- net Net-(Q17-Pad2): track 0.00 -> 5.58 mm
- net Net-(C5-Pad1): track 33.4 -> 28.0 mm
- net Net-(C7-Pad1): track 11.7 -> 6.82 mm
- net Net-(Q6-Pad3): track 5.63 -> 2.32 mm
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- added copper zone on F.Cu, net Net-(C7-Pad2)
Other:
- board outline added: 196.8 x 88.9 mm

Commit message: Primer diseño completo de todo el PCB del amplificador
Parts:
- removed M3: FDS9934C, Package_SO:SOIC-8_3.9x4.9mm_P1.27mm
- removed R100: 680, Resistor_SMD:R_0805_2012Metric_Pad1.15x1.40mm_HandSolder
- added C15: 10u, Capacitor_SMD:C_0805_2012Metric_Pad1.15x1.40mm_HandSolder, F.Cu at (47.0, 78.9)
- added HS1: Heatsink, disipadores:disipador_1.8C, F.Cu at (158.7, 96.2)
- added HS2: Heatsink, disipadores:disipador_5.1C, F.Cu at (95.6, 97.1)
- added J4: Screw_Terminal_01x02, Connector_Phoenix_MC:PhoenixContact_MCV_1,5_2-G-3.5_1x02_P3.50mm_Vertical, F.Cu at (220.4, 98.2)
- added J5: Conn_01x03_Male, Connector_PinHeader_2.54mm:PinHeader_1x03_P2.54mm_Vertical, F.Cu at (36.2, 62.4)
- added J6: Screw_Terminal_01x02, Connector_Phoenix_MC:PhoenixContact_MCV_1,5_2-G-3.5_1x02_P3.50mm_Vertical, F.Cu at (209.4, 56.9)
- added J7: Screw_Terminal_01x02, Connector_Phoenix_MC:PhoenixContact_MCV_1,5_2-G-3.5_1x02_P3.50mm_Vertical, F.Cu at (214.1, 132.6)
- added Q29: BS170, Package_TO_SOT_THT:TO-92_Inline, F.Cu at (221.7, 83.9)
- added R48: 10k, Resistor_SMD:R_0805_2012Metric_Pad1.15x1.40mm_HandSolder, F.Cu at (202.7, 55.9)
- added R52: 0, Resistor_SMD:R_1206_3216Metric_Pad1.42x1.75mm_HandSolder, F.Cu at (52.3, 107.4)
- added R53: 0, Resistor_SMD:R_1206_3216Metric_Pad1.42x1.75mm_HandSolder, F.Cu at (117.8, 134.6)
- added R54: 0, Resistor_SMD:R_1206_3216Metric_Pad1.42x1.75mm_HandSolder, F.Cu at (116.8, 54.8)
- added R55: 0, Resistor_SMD:R_1206_3216Metric_Pad1.42x1.75mm_HandSolder, F.Cu at (126.9, 95.0)
- added R56: 0, Resistor_SMD:R_1206_3216Metric_Pad1.42x1.75mm_HandSolder, F.Cu at (108.6, 96.1)
- added R57: 0, Resistor_SMD:R_1206_3216Metric_Pad1.42x1.75mm_HandSolder, F.Cu at (112.1, 91.1)
- added R59: 0, Resistor_SMD:R_1206_3216Metric_Pad1.42x1.75mm_HandSolder, F.Cu at (139.3, 72.4)
- added R60: 0, Resistor_SMD:R_1206_3216Metric_Pad1.42x1.75mm_HandSolder, F.Cu at (122.3, 82.6)
- added R61: 0, Resistor_SMD:R_1206_3216Metric_Pad1.42x1.75mm_HandSolder, F.Cu at (109.1, 105.0)
- added R62: 0, Resistor_SMD:R_1206_3216Metric_Pad1.42x1.75mm_HandSolder, F.Cu at (112.1, 97.2)
- added R63: 0, Resistor_SMD:R_1206_3216Metric_Pad1.42x1.75mm_HandSolder, F.Cu at (139.2, 69.4)
- added R64: 0, Resistor_SMD:R_1206_3216Metric_Pad1.42x1.75mm_HandSolder, F.Cu at (90.3, 57.3)
- C5, C9: value 10u -> 100u; footprint Capacitor_SMD:C_1206_3216Metric_Pad1.42x1.75mm_HandSolder -> Capacitor_SMD:CP_Elec_8x10.5
- J2: value Conn_01x03_Male -> Screw_Terminal_01x02; footprint Connector_PinHeader_2.54mm:PinHeader_1x03_P2.54mm_Vertical -> Connector_Phoenix_MC:PhoenixContact_MCV_1,5_2-G-3.5_1x02_P3.50mm_Vertical
- J3: value Screw_Terminal_01x06 -> Screw_Terminal_01x02; footprint Connector_Phoenix_MC:PhoenixContact_MCV_1,5_6-G-3.5_1x06_P3.50mm_Vertical -> Connector_Phoenix_MC:PhoenixContact_MCV_1,5_2-G-3.5_1x02_P3.50mm_Vertical
- R29, R33: value 1k -> 10k
- R49: value 600 -> 10k
- moved Q15 208.7 mm to (149.7, 123.6), turned to 90 degrees
- moved R33 196.9 mm to (203.9, 122.7)
- moved R49 191.9 mm to (203.8, 124.9)
- moved Q21 166.8 mm to (125.3, 120.2), turned to 90 degrees
- moved R27 164.3 mm to (145.1, 85.7), turned to 270 degrees
- moved R29 164.0 mm to (202.7, 58.9), turned to 180 degrees
- moved R28 160.6 mm to (144.6, 104.6), turned to 90 degrees
- moved D16 159.6 mm to (88.0, 137.0), turned to 90 degrees
- moved D14 157.5 mm to (125.5, 124.2)
- moved R41 157.4 mm to (62.9, 134.6), turned to 270 degrees
- moved Q13 156.4 mm to (90.5, 105.1), turned to 270 degrees
- moved R39 156.3 mm to (81.8, 122.2)
- moved D10 152.4 mm to (120.5, 107.6), turned to 180 degrees
- moved D11 152.1 mm to (129.9, 119.2), turned to 270 degrees
- moved D12 152.0 mm to (133.0, 119.0), turned to 270 degrees
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Connections:
- C10 pad 1: Earth -> /Vmax
- C10 pad 2: /Vmax -> Earth
- C5 pad 1: Net-(C5-Pad1) -> Earth
- C5 pad 2: Earth -> Net-(C5-Pad2)
- C8 pad 1: /-Vmax -> Earth
- C8 pad 2: Earth -> /-Vmax
- CON1 pad 1: Earth -> Net-(CON1-Pad1)
- CON1 pad 3: Net-(CON1-Pad3) -> Earth
- J1 pad 1: Net-(J1-Pad1) -> /Vmin
- J1 pad 2: Earth -> /Vmax
- J2 pad 1: Net-(C1-Pad2) -> /-Vmax
- J2 pad 2: Net-(J2-Pad2) -> /-Vmin
- J3 pad 1: /Vmin -> Earth
- J3 pad 2: /-Vmin -> Earth
- K1 pad 1: Net-(J1-Pad1) -> Net-(J4-Pad1)
- K1 pad 5: /Vmin -> Net-(K1-Pad5)
- M1 pad 2: Net-(D13-Pad1) -> Net-(M1-Pad2)
- M1 pad 4: Net-(D3-Pad1) -> Net-(M1-Pad4)
- M1 pad 7: Net-(D9-Pad2) -> Net-(M1-Pad7)
- M1 pad 8: Net-(D9-Pad2) -> Net-(M1-Pad7)
- M2 pad 1: Net-(M1-Pad1) -> Net-(M2-Pad1)
- M2 pad 2: Net-(D9-Pad2) -> Net-(M1-Pad7)
- M2 pad 3: Net-(M1-Pad3) -> Net-(M2-Pad3)
- Q11 pad 1: Net-(M1-Pad1) -> Net-(M2-Pad1)
- Q24 pad 2: Net-(D3-Pad1) -> Net-(Q24-Pad2)
- Q25 pad 3: Net-(C5-Pad1) -> Net-(C5-Pad2)
- R10 pad 1: Net-(Q17-Pad2) -> Net-(R10-Pad1)
- R13 pad 1: Net-(Q17-Pad2) -> Net-(R10-Pad1)
- R14 pad 1: Net-(M1-Pad1) -> Net-(M2-Pad1)
- R3 pad 2: Net-(C5-Pad1) -> Net-(C5-Pad2)
- R30 pad 1: Net-(M1-Pad3) -> Net-(M2-Pad3)
- R34 pad 2: Net-(D13-Pad1) -> Net-(M1-Pad2)
- R35 pad 2: /-Vmin -> Net-(R35-Pad2)
- R37 pad 2: /Vmax -> Net-(R37-Pad2)
- R4 pad 2: Net-(C5-Pad1) -> Net-(C5-Pad2)
- R44 pad 2: Net-(C5-Pad1) -> Net-(C5-Pad2)
- R49 pad 1: /Vmin -> /Vmax
- R49 pad 2: Net-(K1-Pad2) -> Net-(D9-Pad2)
- R5 pad 2: /Vmin -> /-Vmin
- R50 pad 2: /Vmin -> Net-(K1-Pad5)
- R7 pad 2: Net-(C5-Pad1) -> Net-(C5-Pad2)
- R8 pad 2: Net-(C5-Pad1) -> Net-(C5-Pad2)
Routing:
- net /VOUT: track 1.77 -> 277.7 mm, vias 1 -> 7
- net Net-(K1-Pad5): track 0.00 -> 191.3 mm
- net Net-(D9-Pad2): track 0.00 -> 187.9 mm
- net Earth: track 24.2 -> 165.8 mm, vias 6 -> 23
- net Net-(D3-Pad1): track 0.00 -> 129.2 mm, vias 0 -> 2
- net /-Vmin: track 0.00 -> 110.6 mm
- net Net-(M1-Pad3): track 0.00 -> 103.6 mm
- net /-Vmax: track 0.00 -> 98.0 mm
- net /Vmax: track 0.00 -> 90.3 mm
- net Net-(C5-Pad2): track 0.00 -> 67.9 mm
- net Net-(M2-Pad1): track 0.00 -> 67.9 mm
- net Net-(Q24-Pad2): track 0.00 -> 63.3 mm
- net Net-(Q17-Pad2): track 5.58 -> 63.0 mm
- net Net-(D21-Pad2): track 0.00 -> 57.3 mm
- net Net-(C6-Pad1): track 19.7 -> 71.9 mm
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- added copper zone on F.Cu, net /-Vmax
- added copper zone on F.Cu, net /-Vmin
- added copper zone on F.Cu, net /VOUT
- added copper zone on F.Cu, net /Vmax
- added copper zone on F.Cu, net /Vmin
- added copper zone on B.Cu, net Earth
- added copper zone on F.Cu, net Earth
- added copper zone on F.Cu, net Net-(D10-Pad1)
- added copper zone on F.Cu, net Net-(D15-Pad1)
- added copper zone on F.Cu, net Net-(D16-Pad2)
- added copper zone on F.Cu, net Net-(D4-Pad2)
Other:
- net class Default: clearance 0.3048 -> 0.4064; trace_width 0.3048 -> 0.4064
- rule trace_clearance: 0.3048 -> 0.4064
